Commit message: Added proper scaling to vehicle model

File: src/vehicle_sim/vehicle/sensor_model/camera/camera_description/urdf/monocular_camera.xacro (robot description, xacro)
@@ -2,6 +2,6 @@
 <robot xmlns:xacro="http://ros.org/wiki/xacro">
   <xacro:property name="pi" value="3.1415926835897931" />
-  <xacro:macro name="monocular_camera_macro" params="suffix parent namespace x y z roll pitch yaw fps width height fov">
-    <xacro:property name="sensor_box" value="0.05" />
+  <xacro:macro name="monocular_camera_macro" params="suffix parent namespace x y z roll pitch yaw fps width height fov scale:=1">
+    <xacro:property name="sensor_box" value="${scale * 0.05}" />
     <xacro:property name="mass" value="0.1" />
     <joint name="${suffix}_joint" type="fixed">

File: src/vehicle_sim/vehicle/sensor_model/imu/imu_description/urdf/imu.xacro (robot description, xacro)
@@ -2,7 +2,7 @@
 <robot xmlns:xacro="http://ros.org/wiki/xacro">
   <xacro:property name="pi" value="3.1415926835897931" />
-  <xacro:macro name="imu_macro" params="suffix parent namespace x y z roll pitch yaw fps">
-    <xacro:property name="sensor_box" value="0.01" />
-    <xacro:property name="mass" value="0.01" />
+  <xacro:macro name="imu_macro" params="suffix parent namespace x y z roll pitch yaw fps scale">
+    <xacro:property name="sensor_box" value="${scale * 0.01}" />
+    <xacro:property name="mass" value="${scale * 0.01}" />
     <joint name="${suffix}_joint" type="fixed">
       <origin rpy="${roll} ${pitch} ${yaw}" xyz="${x} ${y} ${z}"/>

File: src/vehicle_sim/vehicle/sensor_model/velodyne/velodyne_description/urdf/HDL-32E.urdf.xacro (robot description, xacro)
@@ -2,5 +2,5 @@
 <robot xmlns:xacro="http://www.ros.org/wiki/xacro" name="HDL-32E">
   <xacro:property name="M_PI" value="3.1415926535897931" />
-  <xacro:macro name="HDL-32E" params="*origin parent:=base_link name:=velodyne topic:=/velodyne_points organize_cloud:=false hz:=10 lasers:=32 samples:=2187 collision_range:=0.3 min_range:=0.9 max_range:=130.0 noise:=0.008 min_angle:=-${M_PI} max_angle:=${M_PI} gpu:=false">
+  <xacro:macro name="HDL-32E" params="*origin parent:=base_link name:=velodyne topic:=/velodyne_points organize_cloud:=false hz:=10 lasers:=32 samples:=2187 collision_range:=0.3 min_range:=0.9 max_range:=130.0 noise:=0.008 min_angle:=-${M_PI} max_angle:=${M_PI} gpu:=false scale:=1">
     <joint name="${name}_base_mount_joint" type="fixed">
       <xacro:insert_block name="origin" />
@@ -10,6 +10,6 @@
     <link name="${name}_base_link">
       <inertial>
-        <mass value="1.0"/>
-        <origin xyz="0 0 0.07212"/>
+        <mass value="${scale * 1.0}"/>
+        <origin xyz="0 0 ${scale * 0.07212}"/>
         <inertia ixx="${(1.0 * (3.0*0.04267*0.04267 + 0.14424*0.14424)) / 12.0}" ixy="0" ixz="0"
           iyy="${(1.0 * (3.0*0.04267*0.04267 + 0.14424*0.14424)) / 12.0}" iyz="0"
@@ -18,16 +18,16 @@
       <visual>
         <geometry>
-          <mesh filename="package://velodyne_description/meshes/HDL32E_base.dae" />
+          <mesh filename="package://velodyne_description/meshes/HDL32E_base.dae" scale="${scale} ${scale} ${scale}"/>
         </geometry>
       </visual>
       <collision>
-        <origin rpy="0 0 0" xyz="0 0 0.07212"/>
+        <origin rpy="0 0 0" xyz="0 0 ${scale * 0.07212}"/>
         <geometry>
-          <cylinder radius="0.04267" length="0.14424"/>
+          <cylinder radius="${scale * 0.04267}" length="${scale * 0.14424}"/>
         </geometry>
       </collision>
     </link>
     <joint name="${name}_base_scan_joint" type="fixed" >
-      <origin xyz="0 0 0.09081" rpy="0 0 0" />
+      <origin xyz="0 0 ${scale * 0.09081}" rpy="0 0 0" />
       <parent link="${name}_base_link" />
       <child link="${name}"/>
@@ -35,12 +35,12 @@
     <link name="${name}">
       <inertial>
-        <mass value="0.01"/>
+        <mass value="${scale * 0.01}"/>
         <origin xyz="0 0 0"/>
         <inertia ixx="1e-7" ixy="0" ixz="0" iyy="1e-7" iyz="0" izz="1e-7"/>
       </inertial>
       <visual>
-        <origin xyz="0 0 -0.09081" rpy="0 0 0" />
+        <origin xyz="0 0 ${scale * -0.09081}" rpy="0 0 0" />
         <geometry>
-          <mesh filename="package://velodyne_description/meshes/HDL32E_scan.dae" />
+          <mesh filename="package://velodyne_description/meshes/HDL32E_scan.dae" scale="${scale} ${scale} ${scale}"/>
         </geometry>
       </visual>

File: src/vehicle_sim/vehicle/vehicle_model/urdf/body.xacro (robot description, xacro)
@@ -1,5 +1,5 @@
 <?xml version="1.0"?>
 <robot xmlns:xacro="http://ros.org/wiki/xacro">
-  <xacro:macro name="body_macro" params="suffix parent wheel_radius wheel_base vehicle_mass vehicle_mass_height vehicle_width vehicle_length vehicle_height">
+  <xacro:macro name="body_macro" params="suffix parent wheel_radius wheel_base vehicle_mass vehicle_mass_height vehicle_width vehicle_length vehicle_height scale">
   <xacro:property name="pi" value="3.1415926835897931" />
     <joint name="${suffix}_joint" type="fixed">
@@ -24,5 +24,5 @@
         <origin xyz="0 0 0" rpy="0 0 0"/>
         <geometry>
-          <mesh filename="package://vehicle_model/mesh/body.dae" scale="${wheel_base/2.85} 1 1"/>
+          <mesh filename="package://vehicle_model/mesh/body.dae" scale="${wheel_base/2.85} ${scale} ${scale}"/>
         </geometry>
         <material name="black">

File: src/vehicle_sim/vehicle/vehicle_model/urdf/steering.xacro (robot description, xacro)
@@ -1,9 +1,8 @@
 <?xml version="1.0"?>
 <robot xmlns:xacro="http://ros.org/wiki/xacro">
-  <xacro:macro name="steering_macro" params="suffix parent x y yaw length">
+  <xacro:macro name="steering_macro" params="suffix parent x y yaw length scale">
     <xacro:property name="pi" value="3.1415926835897931" />
-    <xacro:property name="radius" value="0.1" />
-    <xacro:property name="length" value="0.01" />
-    <xacro:property name="mass" value="10.0" />
+    <xacro:property name="radius" value="${scale * 0.1}" />
+    <xacro:property name="mass" value="${scale * 10.0}" />
     <joint name="${suffix}_joint" type="revolute">
       <origin rpy="0 0 0" xyz="${x} ${y} 0"/>
@@ -38,9 +37,9 @@
     </link>
   </xacro:macro>
-  <xacro:macro name="steering_link_macro" params="suffix parent x y">
+  <xacro:macro name="steering_link_macro" params="suffix parent x y scale">
     <xacro:property name="pi" value="3.1415926835897931" />
-    <xacro:property name="radius" value="0.1" />
-    <xacro:property name="length" value="0.01" />
-    <xacro:property name="mass" value="10.0" />
+    <xacro:property name="radius" value="${scale * 0.1}" />
+    <xacro:property name="length" value="${scale * 0.01}" />
+    <xacro:property name="mass" value="${scale * 10.0}" />
     <joint name="${suffix}_joint" type="fixed">
       <origin rpy="0 0 0" xyz="${x} ${y} 0"/>

File: src/vehicle_sim/vehicle/vehicle_model/urdf/vehicle.xacro (robot description, xacro)
@@ -9,4 +9,5 @@
   <xacro:include filename="$(find imu_description)/urdf/imu.xacro"/>
   <xacro:arg name="gpu" default="false"/>
+  <xacro:arg name="scale" default="1"/>
   <xacro:property name="pi" value="3.1415926835897931"/>
   <link name="base_footprint"/>
@@ -15,12 +16,13 @@
 	<xacro:property name="vehicle_info" value="${load_yaml('$(find vehicle_model)/config/vehicle_info.yaml')}"/>
   <!-- set parameter -->
-	<xacro:property name="wheel_radius" value="${vehicle_info['wheel_radius']}"/>
-  <xacro:property name="wheel_width" value="${vehicle_info['wheel_width']}"/>
-  <xacro:property name="wheel_base" value="${vehicle_info['wheel_base']}"/>
-  <xacro:property name="wheel_tread" value="${vehicle_info['wheel_tread']}"/>
-  <xacro:property name="vehicle_mass" value="${vehicle_info['vehicle_mass']}"/>
-  <xacro:property name="vehicle_length" value="${vehicle_info['vehicle_length']}"/>
-  <xacro:property name="vehicle_width" value="${vehicle_info['vehicle_width']}"/>
-  <xacro:property name="vehicle_height" value="${vehicle_info['vehicle_height']}"/>
+	<xacro:property name="scale" value="$(arg scale)"/>
+	<xacro:property name="wheel_radius" value="${scale * vehicle_info['wheel_radius']}"/>
+  <xacro:property name="wheel_width" value="${scale * vehicle_info['wheel_width']}"/>
+  <xacro:property name="wheel_base" value="${scale * vehicle_info['wheel_base']}"/>
+  <xacro:property name="wheel_tread" value="${scale * vehicle_info['wheel_tread']}"/>
+  <xacro:property name="vehicle_mass" value="${scale * vehicle_info['vehicle_mass']}"/>
+  <xacro:property name="vehicle_length" value="${scale * vehicle_info['vehicle_length']}"/>
+  <xacro:property name="vehicle_width" value="${scale * vehicle_info['vehicle_width']}"/>
+  <xacro:property name="vehicle_height" value="${scale * vehicle_info['vehicle_height']}"/>
   <xacro:property name="vehicle_mass_height" value="0.5"/>
   <!-- body-->
@@ -33,9 +35,10 @@
                     vehicle_length="${vehicle_length}"
                     vehicle_width="${vehicle_width}"
-                    vehicle_height="${vehicle_height}"/>
+                    vehicle_height="${vehicle_height}"
+                    scale="${scale}"/>
   <!-- steering-->
-  <xacro:steering_link_macro suffix="steering_front" parent="base_link" x="${wheel_base}" y="0"/>
-  <xacro:steering_macro suffix="steering_right_front" parent="steering_front_link" x="0" y="${-1*wheel_tread/2}" yaw="0" length="${wheel_width}"/>
-  <xacro:steering_macro suffix="steering_left_front" parent="steering_front_link" x="0" y="${wheel_tread/2}" yaw="0" length="${wheel_width}"/>
+  <xacro:steering_link_macro suffix="steering_front" parent="base_link" x="${wheel_base}" y="0" scale="${scale}"/>
+  <xacro:steering_macro suffix="steering_right_front" parent="steering_front_link" x="0" y="${-1*wheel_tread/2}" yaw="0" length="${wheel_width}" scale="${scale}"/>
+  <xacro:steering_macro suffix="steering_left_front" parent="steering_front_link" x="0" y="${wheel_tread/2}" yaw="0" length="${wheel_width}" scale="${scale}"/>
   <!-- wheel -->
   <xacro:wheel_macro suffix="wheel_right_front" parent="steering_right_front_link" x="0" y="0" yaw="${pi}" radius="${wheel_radius}" width="${wheel_width}"/>
@@ -49,23 +52,23 @@
   <!-- ================ sensor ================ -->
 	<xacro:property name="calibration" value="${load_yaml('$(find vehicle_model)/config/calibration.yaml')}"/>
-  <xacro:HDL-32E parent="base_link" name="velodyne" topic="/points_raw" hz="10" samples="220" gpu="$(arg gpu)">
-    <origin xyz="${calibration['base_link2velodyne']['x']} ${calibration['base_link2velodyne']['y']} ${calibration['base_link2velodyne']['z']}"
+  <xacro:HDL-32E parent="base_link" name="velodyne" topic="/points_raw" hz="10" samples="220" gpu="$(arg gpu)" scale="${scale}">
+    <origin xyz="${scale * calibration['base_link2velodyne']['x']} ${scale * calibration['base_link2velodyne']['y']} ${scale * calibration['base_link2velodyne']['z']}"
             rpy="${calibration['base_link2velodyne']['roll']} ${calibration['base_link2velodyne']['pitch']} ${calibration['base_link2velodyne']['yaw']}" />
   </xacro:HDL-32E>
   <xacro:monocular_camera_macro suffix="camera" parent="base_link" namespace=""
-                                x="${calibration['base_link2camera']['x']}"
-                                y="${calibration['base_link2camera']['y']}"
-                                z="${calibration['base_link2camera']['z']}"
+                                x="${scale * calibration['base_link2camera']['x']}"
+                                y="${scale * calibration['base_link2camera']['y']}"
+                                z="${scale * calibration['base_link2camera']['z']}"
                                 roll="${calibration['base_link2camera']['roll']}"
                                 pitch="${calibration['base_link2camera']['pitch']}"
                                 yaw="${calibration['base_link2camera']['yaw']}"
-                                fps="30" width="800" height="400" fov="1.3"/>
+                                fps="30" width="800" height="400" fov="1.3" scale="${scale}"/>
   <xacro:imu_macro suffix="imu" parent="base_link" namespace=""
-                   x="${calibration['base_link2imu']['x']}"
-                   y="${calibration['base_link2imu']['y']}"
-                   z="${calibration['base_link2imu']['z']}"
+                   x="${scale * calibration['base_link2imu']['x']}"
+                   y="${scale * calibration['base_link2imu']['y']}"
+                   z="${scale * calibration['base_link2imu']['z']}"
                    roll="${calibration['base_link2imu']['roll']}"
                    pitch="${calibration['base_link2imu']['pitch']}"
                    yaw="${calibration['base_link2imu']['yaw']}"
-                   fps="100" />
+                   fps="100" scale="${scale}"/>
 </robot>
