Commit message: Increased rosbot mass

File: src/vehicle_sim/vehicle_rosbot/urdf/rosbot.xacro (robot description, xacro)
@@ -16,5 +16,5 @@
     <pose>0 0 0.1 0 0 0</pose>
     <inertial>
-      <mass value="5"/>
+      <mass value="35"/>
       <origin xyz="0 0 0.04" rpy=" 0 0 0"/>
       <inertia
@@ -47,5 +47,5 @@
     <pose>0 0 0 0 0 0</pose>
     <inertial>
-      <mass value="0.01"/>
+      <mass value="1"/>
       <origin xyz="0 0 0.055" rpy=" 0 0 0"/>
       <inertia
@@ -87,5 +87,5 @@
     <inertial>
       <origin xyz="0 0 0" rpy="0 1.5707 1.5707"/>
-      <mass value="0.5"/>
+      <mass value="1.5"/>
       <inertia
       ixx="0.001" ixy="0.0" ixz="0.0"
@@ -118,5 +118,5 @@
     <inertial>
       <origin xyz="0 0 0" rpy="0 1.5707 1.5707"/>
-      <mass value="0.5"/>
+      <mass value="1.5"/>
       <inertia
       ixx="0.001" ixy="0.0" ixz="0.0"
@@ -149,5 +149,5 @@
     <inertial>
       <origin xyz="0 0 0" rpy="0 1.5707 1.5707"/>
-      <mass value="0.5"/>
+      <mass value="1.5"/>
       <inertia
       ixx="0.001" ixy="0.0" ixz="0.0"
@@ -180,5 +180,5 @@
     <inertial>
       <origin xyz="0 0 0" rpy="0 1.5707 1.5707"/>
-      <mass value="0.5"/>
+      <mass value="1.5"/>
       <inertia
       ixx="0.001" ixy="0.0" ixz="0.0"
